File: matrix.kicad_sch (KiCad schematic)
At the start: 176 parts

Commit message: 3 viikon muutokset pt2
Parts:
- MX10: value MX-NoLED -> F9
- MX11: value MX-NoLED -> F10
- MX12: value MX-NoLED -> F11
- MX13: value MX-NoLED -> F12
- MX14: value MX-NoLED -> PrtSc
- MX15: value MX-NoLED -> Scroll Lock
- MX16: value MX-NoLED -> Pause Break
- MX17: value MX-NoLED -> §
- MX18: value MX-NoLED -> 1
- MX19: value MX-NoLED -> 2
- MX2: value MX-NoLED -> F1
- MX20: value MX-NoLED -> 3
- MX21: value MX-NoLED -> 4
- MX22: value MX-NoLED -> 5
- MX23: value MX-NoLED -> 6
- MX24: value MX-NoLED -> 7
- MX25: value MX-NoLED -> 8
- MX26: value MX-NoLED -> 9
- MX27: value MX-NoLED -> 0
- MX28: value MX-NoLED -> +
- MX29: value MX-NoLED -> ´
- MX3: value F1 -> F2
- MX30: value MX-NoLED -> Backspace
- MX31: value MX-NoLED -> Insert
- MX32, MX84: value MX-NoLED -> Home
- MX33: value MX-NoLED -> PageUp
- MX34: value MX-NoLED -> Tab
- MX35: value MX-NoLED -> Q
- MX36: value MX-NoLED -> W
- MX37: value MX-NoLED -> E
- MX38: value MX-NoLED -> R
- MX39: value MX-NoLED -> T
- MX4: value F2 -> F3
- MX40: value MX-NoLED -> Y
- MX41: value MX-NoLED -> U
- MX42: value MX-NoLED -> I
- MX43: value MX-NoLED -> O
- MX44: value MX-NoLED -> P
- MX45: value MX-NoLED -> Å
- MX46: value MX-NoLED -> ¨
- MX47: value MX-NoLED -> Delete
- MX48: value MX-NoLED -> End
- MX49: value MX-NoLED -> PageDown
- MX5: value F3 -> F4
- MX50: value MX-NoLED -> CapsLock
- MX51: value MX-NoLED -> A
- MX52: value MX-NoLED -> S
- MX53: value MX-NoLED -> D
- MX54: value MX-NoLED -> F
- MX55: value MX-NoLED -> G
- MX56: value MX-NoLED -> H
- MX57: value MX-NoLED -> J
- MX58: value MX-NoLED -> K
- MX59: value MX-NoLED -> L
- MX6: value F4 -> F5
- MX60: value MX-NoLED -> Ö
- MX61: value MX-NoLED -> Ä
- MX62: value MX-NoLED -> '
- MX63: value MX-NoLED -> Enter
- MX64, MX76: value MX-NoLED -> Shift
- MX65: value MX-NoLED -> <
- MX66: value MX-NoLED -> Z
- MX67: value MX-NoLED -> X
- MX68: value MX-NoLED -> C
- MX69: value MX-NoLED -> V
- MX7: value MX-NoLED -> F6
- MX70: value MX-NoLED -> B
- MX71: value MX-NoLED -> N
- MX72: value MX-NoLED -> M
- MX73: value MX-NoLED -> ,
- MX74: value MX-NoLED -> .
- MX75: value MX-NoLED -> -
- MX77: value MX-NoLED -> UpArrow
- MX78, MX85: value MX-NoLED -> Ctrl
- MX79, MX83: value MX-NoLED -> Win
- MX8: value MX-NoLED -> F7
- MX80: value MX-NoLED -> Alt
- MX81: value MX-NoLED -> Space
- MX82: value MX-NoLED -> Altgr
- MX86: value MX-NoLED -> LeftArrow
- MX87: value MX-NoLED -> DownArrow
- MX88: value MX-NoLED -> RightArrow
- MX9: value MX-NoLED -> F8

Commit message: sch valmis toivottavastipt 2
Parts:
- renumbered D1 to D2, D2 to D3, D3 to D4, D4 to D5

Commit message: Valmis sch pt2
Parts:
- MX1, MX10, MX11, MX12, MX13, MX14, MX15, MX16, MX17, MX18, MX19, MX2, MX20, MX21, MX22, MX23, MX24, MX25, MX26, MX27, MX28, MX29, MX3, MX31, MX32, MX33, MX35, MX36, MX37, MX38, MX39, MX4, MX40, MX41, MX42, MX43, MX44, MX45, MX46, MX47, MX48, MX49, MX5, MX51, MX52, MX53, MX54, MX55, MX56, MX57, MX58, MX59, MX6, MX60, MX61, MX62, MX65, MX66, MX67, MX68, MX69, MX7, MX70, MX71, MX72, MX73, MX74, MX75, MX77, MX8, MX86, MX87, MX88, MX9: footprint MX_Alps_Hybrid:MX-1U-NoLED -> Alps_Only:ALPS-1U
- MX30: footprint MX_Alps_Hybrid:MX-1U-NoLED -> Alps_Only:ALPS-2U
- MX34: footprint MX_Alps_Hybrid:MX-1U-NoLED -> Alps_Only:ALPS-1.5U
- MX50: footprint MX_Alps_Hybrid:MX-1U-NoLED -> Alps_Only:ALPS-1.75U
- MX63: footprint MX_Alps_Hybrid:MX-1U-NoLED -> Alps_Only:ALPS-ISO
- MX64, MX78, MX79, MX80, MX82, MX83, MX85: footprint MX_Alps_Hybrid:MX-1U-NoLED -> Alps_Only:ALPS-1.25U
- MX76: footprint MX_Alps_Hybrid:MX-1U-NoLED -> Alps_Only:ALPS-2.75U
- MX81: footprint MX_Alps_Hybrid:MX-1U-NoLED -> Alps_Only:ALPS-6.25U
- MX84: value Home -> Menu; footprint MX_Alps_Hybrid:MX-1U-NoLED -> Alps_Only:ALPS-1.25U
