File: oikeanappis.kicad_sch (KiCad schematic)
At the start: 20 parts, among them J1 AVR-ISP-6, SW1 SW_Push, U1 ATmega32U4-A, Y1 16MHz

Commit message: sch valmis toivottavastipt 2
Parts:
- removed J1: AVR-ISP-6, symbol Connector:AVR-ISP-6
- C1: renamed from C7; footprint Capacitor_SMD:C_0805_2012Metric -> Capacitor_SMD:C_0805_2012Metric_Pad1.18x1.45mm_HandSolder
- C2: renamed from C6; footprint Capacitor_SMD:C_0805_2012Metric -> Capacitor_SMD:C_0805_2012Metric_Pad1.18x1.45mm_HandSolder
- C3: renamed from C1; footprint Capacitor_SMD:C_0805_2012Metric -> Capacitor_SMD:C_0805_2012Metric_Pad1.18x1.45mm_HandSolder
- C4: renamed from C2; footprint Capacitor_SMD:C_0805_2012Metric -> Capacitor_SMD:C_0805_2012Metric_Pad1.18x1.45mm_HandSolder
- C5: renamed from C3; footprint Capacitor_SMD:C_0805_2012Metric -> Capacitor_SMD:C_0805_2012Metric_Pad1.18x1.45mm_HandSolder
- C6: renamed from C4; footprint Capacitor_SMD:C_0805_2012Metric -> Capacitor_SMD:C_0805_2012Metric_Pad1.18x1.45mm_HandSolder
- C7: renamed from C5; footprint Capacitor_SMD:C_0805_2012Metric -> Capacitor_SMD:C_0805_2012Metric_Pad1.18x1.45mm_HandSolder
- renumbered D5 to D1, R4 to R1, R1 to R2, R2 to R3, R3 to R4
Connections:
- net COL7: now reaches U1.12 (PB7)
- net COL10: now reaches U1.18 (PD0)
- net COL11: now reaches U1.19 (PD1)
- net COL12: now reaches U1.20 (PD2)
- net COL13: now reaches U1.21 (PD3)
- net COL15: now reaches U1.22 (PD5)
- net COL14: now reaches U1.25 (PD4)
- net COL16: now reaches U1.26 (PD6)
- net COL4: now reaches U1.28 (PB4)
- net COL5: now reaches U1.29 (PB5)
- net COL6: now reaches U1.30 (PB6)
- net COL8: now reaches U1.31 (PC6)
- net COL9: now reaches U1.32 (PC7)
- net ROW5: now reaches U1.36 (PF7)
- net ROW4: now reaches U1.37 (PF6)
- net ROW3: now reaches U1.38 (PF5)
- net ROW2: now reaches U1.39 (PF4)
- net ROW1: now reaches U1.40 (PF1)
- net ROW0: now reaches U1.41 (PF0)
- net COL0: now reaches U1.8 (PB0)
- net MISO renamed COL3
- net MOSI renamed COL2
- net SCK renamed COL1

Commit message: Valmis sch pt2
Parts:
- D1: footprint Package_TO_SOT_SMD:SOT-143 -> Fuse:Fuse_1206_3216Metric_Pad1.42x1.75mm_HandSolder
- F1: footprint (none) -> Fuse:Fuse_1206_3216Metric_Pad1.42x1.75mm_HandSolder
- R1, R2: footprint Resistor_SMD:R_0805_2012Metric -> Resistor_SMD:R_0805_2012Metric_Pad1.20x1.40mm_HandSolder
- R3, R4: value 22k -> 22; footprint (none) -> Resistor_SMD:R_0805_2012Metric_Pad1.20x1.40mm_HandSolder
- R5, R6: footprint (none) -> Resistor_SMD:R_0805_2012Metric_Pad1.20x1.40mm_HandSolder
- USB1: footprint (none) -> Alps_Only:ALPS-2U
Connections:
- net D+: now also R4.2; no longer R3.1
- net D-: now also R3.1; no longer R4.2
- no-connect marks 0 -> 5
Changed lines of the file:
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@@
   (junction (at 43.18 97.79) (diameter 0) (color 0 0 0 0)
   )
+  (no_connect (at 72.39 55.88))
+  (no_connect (at 102.87 96.52))
+  (no_connect (at 41.91 157.48))
+  (no_connect (at 41.91 142.24))
+  (no_connect (at 102.87 88.9))
   (wire (pts (xy 41.91 167.64) (xy 44.45 167.64))
     (stroke (width 0) (type default))
@@
     )
   )
-  (global_label "D+" (shape input) (at 93.98 152.4 0) (fields_autoplaced)
+  (global_label "D-" (shape input) (at 93.98 152.4 0) (fields_autoplaced)
     (effects (font (size 1.27 1.27)) (justify left))
     (property "Intersheetrefs" "${INTERSHEET_REFS}" (at 99.8076 152.4 0)
@@
     )
   )
-  (global_label "D-" (shape input) (at 93.98 154.94 0) (fields_autoplaced)
+  (global_label "D+" (shape input) (at 93.98 154.94 0) (fields_autoplaced)
     (effects (font (size 1.27 1.27)) (justify left))
     (property "Intersheetrefs" "${INTERSHEET_REFS}" (at 99.8076 154.94 0)
@@
       (effects (font (size 1.27 1.27)))
     )
-    (property "Footprint" "Resistor_SMD:R_0805_2012Metric" (at 111.76 93.98 0)
+    (property "Footprint" "Resistor_SMD:R_0805_2012Metric_Pad1.20x1.40mm_HandSolder" (at 111.76 93.98 0)
       (effects (font (size 1.27 1.27)) hide)
     )
@@
       (effects (font (size 1.524 1.524)))
     )
-    (property "Footprint" "" (at 39.37 151.13 0)
+    (property "Footprint" "Alps_Only:ALPS-2U" (at 39.37 151.13 0)
       (effects (font (size 1.524 1.524)) hide)
     )
@@
       (effects (font (size 1.27 1.27)) (justify right))
     )
-    (property "Footprint" "Resistor_SMD:R_0805_2012Metric" (at 71.12 35.56 0)
+    (property "Footprint" "Resistor_SMD:R_0805_2012Metric_Pad1.20x1.40mm_HandSolder" (at 71.12 35.56 0)
       (effects (font (size 1.27 1.27)) hide)
     )
@@
       (effects (font (size 1.27 1.27)))
     )
-    (property "Footprint" "Package_TO_SOT_SMD:SOT-143" (at 85.09 168.656 0)
+    (property "Footprint" "Fuse:Fuse_1206_3216Metric_Pad1.42x1.75mm_HandSolder" (at 85.09 168.656 0)
       (effects (font (size 1.27 1.27)) hide)
     )
@@
   )
   (symbol (lib_id "power:PWR_FLAG") (at 59.69 139.7 0) (unit 1)
-    (in_bom yes) (on_board yes) (dnp no) (fields_autoplaced)
+    (in_bom yes) (on_board yes) (dnp no)
     (property "Reference" "#FLG02" (at 59.69 137.795 0)
       (effects (font (size 1.27 1.27)) hide)
     )
-    (property "Value" "PWR_FLAG" (at 59.69 134.62 0)
+    (property "Value" "PWR_FLAG" (at 64.77 132.08 0)
       (effects (font (size 1.27 1.27)))
     )
@@
       (effects (font (size 1.27 1.27)))
     )
-    (property "Value" "22k" (at 90.17 149.86 90)
-      (effects (font (size 1.27 1.27)))
-    )
-    (property "Footprint" "" (at 90.17 152.4 0)
+    (property "Value" "22" (at 90.17 149.86 90)
+      (effects (font (size 1.27 1.27)))
+    )
+    (property "Footprint" "Resistor_SMD:R_0805_2012Metric_Pad1.20x1.40mm_HandSolder" (at 90.17 152.4 0)
       (effects (font (size 1.27 1.27)) hide)
     )
@@
       (effects (font (size 1.27 1.27)) (justify left))
     )
-    (property "Footprint" "" (at 62.23 162.56 0)
+    (property "Footprint" "Resistor_SMD:R_0805_2012Metric_Pad1.20x1.40mm_HandSolder" (at 62.23 162.56 0)
       (effects (font (size 1.27 1.27)) hide)
     )
@@
       (effects (font (size 1.27 1.27)) (justify left))
     )
-    (property "Footprint" "" (at 57.15 162.56 0)
+    (property "Footprint" "Resistor_SMD:R_0805_2012Metric_Pad1.20x1.40mm_HandSolder" (at 57.15 162.56 0)
       (effects (font (size 1.27 1.27)) hide)
     )
@@
       (effects (font (size 1.27 1.27)))
     )
-    (property "Value" "22k" (at 90.17 158.75 90)
-      (effects (font (size 1.27 1.27)))
-    )
-    (property "Footprint" "" (at 90.17 154.94 0)
+    (property "Value" "22" (at 90.17 158.75 90)
+      (effects (font (size 1.27 1.27)))
+    )
+    (property "Footprint" "Resistor_SMD:R_0805_2012Metric_Pad1.20x1.40mm_HandSolder" (at 90.17 154.94 0)
       (effects (font (size 1.27 1.27)) hide)
     )
@@
   (symbol (lib_id "Device:Polyfuse_Small") (at 55.88 139.7 90) (unit 1)
     (in_bom yes) (on_board yes) (dnp no)
-    (property "Reference" "F1" (at 59.69 133.35 90)
-      (effects (font (size 1.27 1.27)))
-    )
-    (property "Value" "Polyfuse_Small" (at 59.69 135.89 90)
-      (effects (font (size 1.27 1.27)))
-    )
-    (property "Footprint" "" (at 60.96 138.43 0)
-      (effects (font (size 1.27 1.27)) (justify left) hide)
-    )
+    (property "Reference" "F1" (at 55.88 132.08 90)
+      (effects (font (size 1.27 1.27)))
+    )
+    (property "Value" "Polyfuse_Small" (at 58.42 135.89 90)
+      (effects (font (size 1.27 1.27)))
+    )
+    (property "Footprint" "Fuse:Fuse_1206_3216Metric_Pad1.42x1.75mm_HandSolder" (at 60.96 138.43 0)
+      (effects (font (size 1.27 1.27)) (justify left) hide)
+    )
